File: chocobanan.kicad_pcb (KiCad board)
At the start: 2 copper layers, 270.8 x 113.3 mm, 131 parts, among them SW1 SW_DIP_x01, SW49 Rotary_Encoder_Switch, U1 Elite-C

Commit message: start pcb
Parts:
- removed D49, D50, D51, D52, D53, D54, D55, D58, D59: D_Small, keebio-parts:Diode_Long
- removed D56, D57: LED, keebio-parts:LED_3mm
- removed MX49, MX50, MX51, MX52, MX53, MX56, MX58, MX59: MX-NoLED, MX_Only:MXOnly-1U-Hotswap
- removed MX54: MX-NoLED, MX_Only:MXOnly-1.5U-Hotswap
- removed MX55, MX57: MX-NoLED, MX_Only:MXOnly-1.25U-Hotswap
- removed MX60: MX-NoLED, MX_Only:MXOnly-2.25U-Hotswap-ReversedStabilizers
- removed MX61: MX-NoLED, MX_Only:MXOnly-2.75U-Hotswap-ReversedStabilizers
- removed R1, R2: R_Small, keebio-parts:Resistor-Compact-1-side
- removed REF** (x6): MountingHole_2.2mm_M2, MountingHole:MountingHole_2.2mm_M2
- removed SW1: SW_DIP_x01, kbd:ResetSW_4P
- D1, D10, D11, D12, D13, D14, D15, D16, D17, D18, D19, D2, D20, D21, D22, D23, D24, D25, D26, D27, D28, D29, D3, D30, D31, D32, D33, D34, D35, D36, D37, D38, D39, D4, D40, D41, D42, D43, D44, D45, D46, D47, D48, D5, D6, D7, D8, D9: footprint keebio-parts:Diode_Long -> kbd:D3_TH_SMD_only_back; moved to F.Cu
- MX1: footprint MX_Only:MXOnly-1U-Hotswap -> MX_Only:MXOnly-1.5U-NoLED
- MX10, MX11, MX13, MX14, MX15, MX17, MX18, MX19, MX21, MX22, MX23, MX24, MX25, MX26, MX27, MX28, MX29, MX30, MX31, MX32, MX33, MX34, MX35, MX36, MX37, MX38, MX39, MX40, MX41, MX42, MX43, MX44, MX45, MX46, MX47, MX48, MX5, MX6, MX7, MX9: footprint MX_Only:MXOnly-1U-Hotswap -> MX_Only:MXOnly-1U-NoLED
- MX12, MX8: footprint MX_Only:MXOnly-1U-Hotswap -> MX_Only:MXOnly-1.25U-NoLED
- MX16: footprint MX_Only:MXOnly-1U-Hotswap -> MX_Only:MXOnly-2.25U-NoLED
- MX2: footprint MX_Only:MXOnly-1.5U-Hotswap -> MX_Only:MXOnly-1.75U-NoLED
- MX20: footprint MX_Only:MXOnly-6.25U-Hotswap -> MX_Only:MXOnly-2U-NoLED
- MX3: footprint MX_Only:MXOnly-1.75U-Hotswap -> MX_Only:MXOnly-2.25U-NoLED
- MX4: footprint MX_Only:MXOnly-2.25U-Hotswap -> MX_Only:MXOnly-1.25U-NoLED
- SW49: moved to F.Cu
- U1: value Elite-C -> ProMicro; footprint keebio-parts:Elite-C -> keebio-parts:ArduinoProMicro
- moved D26 263.0 mm to (351.0, 121.9), turned to 0 degrees
- moved D28 261.3 mm to (371.0, 111.3), turned to 0 degrees
- moved D31 252.5 mm to (361.0, 116.6), turned to 0 degrees
- moved D27 252.4 mm to (341.0, 132.5), turned to 0 degrees
- moved D24 248.4 mm to (351.0, 119.2), turned to 0 degrees
- moved D32 247.8 mm to (361.0, 119.2), turned to 0 degrees
- moved MX27 246.9 mm to (350.7, 45.0)
- moved D36 241.2 mm to (371.0, 113.9), turned to 0 degrees
- moved D20 237.1 mm to (351.0, 116.6), turned to 0 degrees
- moved D33 229.3 mm to (351.0, 127.2), turned to 0 degrees
- moved D37 227.4 mm to (351.0, 132.5), turned to 0 degrees
- moved D29 225.0 mm to (341.0, 135.1), turned to 0 degrees
- moved D41 223.0 mm to (361.0, 129.8), turned to 0 degrees
- moved D38 219.0 mm to (361.0, 121.9), turned to 0 degrees
- moved D42 212.3 mm to (351.0, 135.1), turned to 0 degrees
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Connections:
- net rowMX57 renamed Net-(D5-Pad2)
- net rowMX58 renamed Net-(D10-Pad2)
- net rowMX59 renamed Net-(D15-Pad2)
- D1 pad 1: row0 -> Net-(D1-Pad1)
- D10 pad 1: row4 -> Net-(D10-Pad1)
- D11 pad 1: row0 -> Net-(D11-Pad1)
- D12 pad 1: row1 -> Net-(D12-Pad1)
- D13 pad 1: row2 -> Net-(D1-Pad1)
- D14 pad 1: row3 -> Net-(D10-Pad1)
- D15 pad 1: row4 -> Net-(D11-Pad1)
- D16 pad 1: row0 -> Net-(D12-Pad1)
- D17 pad 1: row1 -> Net-(D1-Pad1)
- D18 pad 1: row2 -> Net-(D10-Pad1)
- D19 pad 1: row3 -> Net-(D11-Pad1)
- D2 pad 1: row1 -> Net-(D10-Pad1)
- D20 pad 1: row4 -> Net-(D12-Pad1)
- D21 pad 1: row0 -> Net-(D1-Pad1)
- D22 pad 1: row1 -> Net-(D10-Pad1)
- D23 pad 1: row2 -> Net-(D11-Pad1)
- D24 pad 1: row3 -> Net-(D12-Pad1)
- D24 pad 2: Net-(D24-Pad2) -> enc_pin2
- D25 pad 1: row4 -> Net-(D1-Pad1)
- D26 pad 1: row0 -> Net-(D10-Pad1)
- D27 pad 1: row1 -> Net-(D11-Pad1)
- D28 pad 1: row2 -> Net-(D12-Pad1)
- D29 pad 1: row3 -> Net-(D1-Pad1)
- D3 pad 1: row2 -> Net-(D11-Pad1)
- D30 pad 1: row4 -> Net-(D10-Pad1)
- D31 pad 1: row0 -> Net-(D11-Pad1)
- D32 pad 1: row1 -> Net-(D12-Pad1)
- D33 pad 1: row2 -> Net-(D1-Pad1)
- D34 pad 1: row3 -> Net-(D10-Pad1)
- D35 pad 1: row4 -> Net-(D11-Pad1)
- D36 pad 1: row0 -> Net-(D12-Pad1)
- D37 pad 1: row1 -> Net-(D1-Pad1)
- D38 pad 1: row2 -> Net-(D10-Pad1)
- D39 pad 1: row3 -> Net-(D11-Pad1)
- D4 pad 1: row3 -> Net-(D12-Pad1)
- D40 pad 1: row4 -> Net-(D12-Pad1)
- D41 pad 1: row0 -> Net-(D1-Pad1)
- D42 pad 1: row1 -> Net-(D10-Pad1)
- D43 pad 1: row2 -> Net-(D11-Pad1)
- D44 pad 1: row3 -> Net-(D12-Pad1)
- D45 pad 1: row0 -> Net-(D1-Pad1)
- D46 pad 1: row1 -> Net-(D10-Pad1)
- D47 pad 1: row2 -> Net-(D11-Pad1)
- D48 pad 1: row3 -> Net-(D12-Pad1)
- D5 pad 1: row4 -> Net-(D1-Pad1)
- D6 pad 1: row0 -> Net-(D10-Pad1)
- D7 pad 1: row1 -> Net-(D11-Pad1)
- D8 pad 1: row2 -> Net-(D12-Pad1)
- D9 pad 1: row3 -> Net-(D1-Pad1)
- MX10 pad 1: col1 -> col2
- MX13 pad 1: col2 -> col3
- MX14 pad 1: col2 -> col3
- MX15 pad 1: col2 -> col3
- MX17 pad 1: col3 -> col4
- MX18 pad 1: col3 -> col4
- MX19 pad 1: col3 -> col4
- MX21 pad 1: col4 -> col5
- MX22 pad 1: col4 -> col5
- MX23 pad 1: col4 -> col5
- MX24 pad 1: col4 -> col5
- MX24 pad 2: Net-(D24-Pad2) -> enc_pin2
- MX25 pad 1: col8 -> col6
- MX26 pad 1: col5 -> col6
- MX27 pad 1: col5 -> col6
- MX28 pad 1: col5 -> col6
- MX29 pad 1: col5 -> col7
- MX30 pad 1: col9 -> col7
- MX31 pad 1: col6 -> col7
- MX32 pad 1: col6 -> col7
- MX33 pad 1: col6 -> col8
- MX34 pad 1: col6 -> col8
- MX35 pad 1: col10 -> col8
- MX36 pad 1: col7 -> col8
- MX37 pad 1: col7 -> col9
- MX38 pad 1: col7 -> col9
- MX39 pad 1: col7 -> col9
- MX40 pad 1: col11 -> col9
- MX41 pad 1: col8 -> col10
- MX42 pad 1: col8 -> col10
- MX43 pad 1: col8 -> col10
- MX44 pad 1: col8 -> col10
- MX45 pad 1: col9 -> col11
- MX46 pad 1: col9 -> col11
- MX47 pad 1: col9 -> col11
- MX48 pad 1: col9 -> col11
- MX5 pad 1: col0 -> col1
- MX9 pad 1: col1 -> col2
- SW49 pad S1: switchpin1 -> col5
- SW49 pad S2: col11 -> enc_pin2
- U1 pad 1: Net-(U1-Pad1) -> rot1
- U1 pad 10: row0 -> Net-(U1-Pad10)
- U1 pad 11: CapsLed -> Net-(U1-Pad11)
- U1 pad 12: LayerLed -> Net-(U1-Pad12)
- U1 pad 13: col4 -> Net-(U1-Pad13)
- U1 pad 14: col5 -> Net-(U1-Pad14)
- U1 pad 15: col6 -> Net-(U1-Pad15)
- U1 pad 16: col7 -> Net-(U1-Pad16)
- U1 pad 17: col8 -> Net-(U1-Pad17)
- U1 pad 18: col9 -> Net-(U1-Pad18)
- U1 pad 19: col10 -> Net-(U1-Pad19)
- U1 pad 2: Net-(U1-Pad2) -> rot0
- U1 pad 20: col11 -> Net-(U1-Pad20)
- U1 pad 22: RST -> Net-(U1-Pad22)
- U1 pad 23: GND -> Net-(U1-Pad23)
- U1 pad 24: col0 -> Net-(U1-Pad24)
- U1 pad 3: GND -> Net-(U1-Pad3)
- U1 pad 4: GND -> Net-(U1-Pad4)
- U1 pad 6: row4 -> Net-(U1-Pad6)
- U1 pad 7: row3 -> Net-(U1-Pad7)
- U1 pad 8: row2 -> Net-(U1-Pad8)
- U1 pad 9: row1 -> Net-(U1-Pad9)
Routing:
- net row2: track 375.7 -> 0.00 mm
- net row3: track 370.6 -> 0.00 mm
- net row4: track 364.7 -> 0.00 mm
- net col11: track 354.5 -> 0.00 mm
- net row0: track 323.5 -> 0.00 mm
- net col10: track 313.8 -> 0.00 mm
- net row1: track 305.1 -> 0.00 mm
- net col9: track 291.2 -> 0.00 mm
- net col8: track 261.2 -> 0.00 mm
- net LayerLed: track 253.8 -> 0.00 mm
- net rot1: track 239.7 -> 0.00 mm
- net rot0: track 233.5 -> 0.00 mm
- net CapsLed: track 230.5 -> 0.00 mm
- net col6: track 220.8 -> 0.00 mm
- net col7: track 207.1 -> 0.00 mm
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Other:
- board outline removed
- board text removed: "+"
- board text removed: "-"

Commit message: clean up and technical drawings pcb
Parts:
- U1: footprint keebio-parts:ArduinoProMicro -> kbd:ArduinoProMicro_centered
- moved D20 245.5 mm to (109.9, 70.2), turned to 80 degrees
- moved U1 187.9 mm to (23.9, -26.4), turned to 270 degrees
Routing:
- net Net-(D10-Pad1): track 98.5 -> 51.2 mm
- net Net-(D1-Pad1): track 97.9 -> 51.2 mm
- net Net-(D11-Pad1): track 95.7 -> 50.5 mm
- net Net-(D23-Pad2): track 12.8 -> 2.04 mm
- net Net-(D22-Pad2): track 12.8 -> 2.04 mm
- net Net-(D21-Pad2): track 12.8 -> 2.04 mm
- net Net-(D15-Pad2): track 12.8 -> 2.04 mm
- net Net-(D14-Pad2): track 12.8 -> 2.04 mm
- net Net-(D13-Pad2): track 12.8 -> 2.04 mm
- net Net-(D12-Pad2): track 10.6 -> 2.04 mm
- net Net-(D1-Pad2): track 19.2 -> 12.7 mm
- net Net-(D19-Pad2): track 8.04 -> 2.04 mm
- net Net-(D18-Pad2): track 8.04 -> 2.04 mm
- net Net-(D17-Pad2): track 8.04 -> 2.04 mm
- net Net-(D10-Pad2): track 8.04 -> 2.04 mm
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