File: chocobanan.kicad_pcb (KiCad board)
At the start: 2 copper layers, 158.9 x 92.3 mm, 59 parts, among them SW1 RotaryEncoder_Switch, U1 ProMicro, U2 TRRS, U3 Pimoroni_trackpoint

Commit message: clean up
Parts:
- removed MX25: MX-NoLED, MX_Only:MXOnly-2U-ReversedStabilizers-NoLED
- added H1: MountingHole, MountingHole:MountingHole_2.1mm, F.Cu at (-12.8, -8.04)
- added H2: MountingHole, MountingHole:MountingHole_2.1mm, F.Cu at (-17.6, 65.2)
- added H3: MountingHole, MountingHole:MountingHole_2.1mm, F.Cu at (110.0, 3.77)
- added H4: MountingHole, MountingHole:MountingHole_2.1mm, F.Cu at (133.5, 46.6)
- added H5: MountingHole, MountingHole:MountingHole_2.1mm, F.Cu at (127.4, 81.2)
- added MX12.1: MX-NoLED, MX_Only:MXOnly-1U-NoLED, F.Cu at (59.9, 61.1)
- added MX2.1: MX-NoLED, MX_Only:MXOnly-1.25U-NoLED, F.Cu at (-7.14, 19.1)
- added MX20.1: MX-NoLED, MX_Only:MXOnly-2U-ReversedStabilizers-NoLED, F.Cu at (122.5, 62.5)
- added MX8.1: MX-NoLED, MX_Only:MXOnly-1U-NoLED, F.Cu at (14.3, 57.1)
- U1: footprint kbd:ArduinoProMicro_centered -> Custom_footprints_Léon:ArduinoProMicro_centered
- turned U1 to 0 degrees
Routing:
- net COL5: track 68.8 -> 140.4 mm
- net VCC: track 322.4 -> 377.0 mm, vias 6 -> 7
- net ROW3_L: track 125.4 -> 178.9 mm
- net COL4: track 95.8 -> 149.1 mm
- net Net-(RGB1-Pad2): track 4.00 -> 56.9 mm, vias 2 -> 3
- net COL1: track 45.0 -> 84.4 mm, vias 0 -> 1
- net COL3: track 80.2 -> 116.3 mm
- net ROW0_L: track 71.4 -> 102.9 mm
- net ROW2_L: track 91.5 -> 120.5 mm
- net COL0: track 60.1 -> 87.8 mm
- net ROW1_L: track 70.3 -> 93.2 mm
- net COL2: track 66.8 -> 87.9 mm
- net RGB: track 2.00 -> 22.0 mm
- net Net-(D2-Pad2): track 15.7 -> 20.4 mm
- net Net-(D20-Pad2): track 17.0 -> 21.6 mm
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Other:
- board text added: "Chocobanan V1.0"
- board text added: "Designed by Léon Ratinckx(Leonrat#4149)"
- board text added: "Idea by ItsMart06#0380"
