File: chocobanan.sch (KiCad schematic (older format))
At the start: 125 parts, among them SW1 SW_DIP_x01, SW49 Rotary_Encoder_Switch, U1 Elite-C

Commit message: start pcb
Parts:
- removed D49, D50, D51, D52, D53, D54, D55, D58, D59: D_Small, keebio-parts:Diode_Long, symbol Device:D_Small
- removed D56, D57: LED, keebio-parts:LED_3mm, symbol Device:LED
- removed MX49, MX50, MX51, MX52, MX53, MX56, MX58, MX59: MX-NoLED, MX_Only:MXOnly-1U-Hotswap, symbol MX_Alps_Hybrid:MX-NoLED
- removed MX54: MX-NoLED, MX_Only:MXOnly-1.5U-Hotswap, symbol MX_Alps_Hybrid:MX-NoLED
- removed MX55, MX57: MX-NoLED, MX_Only:MXOnly-1.25U-Hotswap, symbol MX_Alps_Hybrid:MX-NoLED
- removed MX60: MX-NoLED, MX_Only:MXOnly-2.25U-Hotswap-ReversedStabilizers, symbol MX_Alps_Hybrid:MX-NoLED
- removed MX61: MX-NoLED, MX_Only:MXOnly-2.75U-Hotswap-ReversedStabilizers, symbol MX_Alps_Hybrid:MX-NoLED
- removed R1, R2: R_Small, keebio-parts:Resistor, symbol Device:R_Small
- removed SW1: SW_DIP_x01, kbd:ResetSW_4P, symbol Switch:SW_DIP_x01
- removed U1: Elite-C, keebio-parts:Elite-C, symbol keebio:Elite-C
- added U1: ProMicro, keebio-parts:ArduinoProMicro, symbol keebio:ProMicro
- D1, D10, D11, D12, D13, D14, D15, D16, D17, D18, D19, D2, D20, D21, D22, D23, D24, D25, D26, D27, D28, D29, D3, D30, D31, D32, D33, D34, D35, D36, D37, D38, D39, D4, D40, D41, D42, D43, D44, D45, D46, D47, D48, D5, D6, D7, D8, D9: footprint keebio-parts:Diode_Long -> kbd:D3_TH_SMD_only_back
- MX1: footprint MX_Only:MXOnly-1U-Hotswap -> MX_Only:MXOnly-1.5U-NoLED
- MX10, MX11, MX13, MX14, MX15, MX17, MX18, MX19, MX21, MX22, MX23, MX24, MX25, MX26, MX27, MX28, MX29, MX30, MX31, MX32, MX33, MX34, MX35, MX36, MX37, MX38, MX39, MX40, MX41, MX42, MX43, MX44, MX45, MX46, MX47, MX48, MX5, MX6, MX7, MX9: footprint MX_Only:MXOnly-1U-Hotswap -> MX_Only:MXOnly-1U-NoLED
- MX12, MX8: footprint MX_Only:MXOnly-1U-Hotswap -> MX_Only:MXOnly-1.25U-NoLED
- MX16: footprint MX_Only:MXOnly-1U-Hotswap -> MX_Only:MXOnly-2.25U-NoLED
- MX2: footprint MX_Only:MXOnly-1.5U-Hotswap -> MX_Only:MXOnly-1.75U-NoLED
- MX20: footprint MX_Only:MXOnly-6.25U-Hotswap -> MX_Only:MXOnly-2U-NoLED
- MX3: footprint MX_Only:MXOnly-1.75U-Hotswap -> MX_Only:MXOnly-2.25U-NoLED
- MX4: footprint MX_Only:MXOnly-2.25U-Hotswap -> MX_Only:MXOnly-1.25U-NoLED
Connections:
- net labels added: enc_pin1, enc_pin2
- net labels removed: CapsLed, LayerLed, RST, row0, row1, row2, row3, row4, rowMX57, rowMX58, rowMX59, switchpin1, switchpin2
- wire segments 165 -> 128
Other:
- moved on the sheet: SW49

Commit message: clean up and technical drawings pcb
Parts:
- U1: footprint keebio-parts:ArduinoProMicro -> kbd:ArduinoProMicro_centered
Changed lines of the file:
@@
 F 0 "U1" H 1700 2987 60  0000 C CNN
 F 1 "ProMicro" H 1700 2881 60  0000 C CNN
-F 2 "keebio-parts:ArduinoProMicro" V 2750 -350 60  0001 C CNN
+F 2 "kbd:ArduinoProMicro_centered" V 2750 -350 60  0001 C CNN
 F 3 "" V 2750 -350 60  0001 C CNN
 	1    1700 2150
