File: chocobanan.kicad_sch (KiCad schematic)
At the start: 48 parts

Commit message: safety push
Parts:
- removed D? (x24): D_Small, symbol Device:D_Small
- removed SW? (x24): SW_PUSH, symbol kbd:SW_PUSH
- added D1, D10, D11, D12, D13, D14, D15, D16, D17, D18, D19, D2, D20, D21, D22, D23, D24, D3, D4, D5, D6, D7, D8, D9: D_Small, kbd:D3_TH_SMD_only_back, symbol Device:D_Small
- added MX1: MX-NoLED, MX_Only:MXOnly-1.5U-NoLED, symbol MX_Alps_Hybrid:MX-NoLED
- added MX10, MX11, MX13, MX14, MX15, MX17, MX18, MX19, MX20, MX21, MX22, MX23, MX24, MX5, MX6, MX7, MX9: MX-NoLED, MX_Only:MXOnly-1U-NoLED, symbol MX_Alps_Hybrid:MX-NoLED
- added MX12, MX4, MX8: MX-NoLED, MX_Only:MXOnly-1.25U-NoLED, symbol MX_Alps_Hybrid:MX-NoLED
- added MX16: MX-NoLED, MX_Only:MXOnly-2.25U-ReversedStabilizers-NoLED, symbol MX_Alps_Hybrid:MX-NoLED
- added MX2: MX-NoLED, MX_Only:MXOnly-1.75U-NoLED, symbol MX_Alps_Hybrid:MX-NoLED
- added MX25: MX-NoLED, MX_Only:MXOnly-2U-ReversedStabilizers-NoLED, symbol MX_Alps_Hybrid:MX-NoLED
- added MX3: MX-NoLED, MX_Only:MXOnly-2.25U-NoLED, symbol MX_Alps_Hybrid:MX-NoLED
- added RGB1, RGB2, RGB3, RGB4, RGB5, RGB6: WS2812B, kbd:LED_WS2812B-PLCC4, symbol LED:WS2812B
- added SW1: RotaryEncoder_Switch, Custom_footprints_Léon:RotaryEncoder_EC11_Switch, symbol Device:RotaryEncoder_Switch
- added U1: ProMicro, kbd:ArduinoProMicro_centered, symbol kbd:ProMicro
- added U2: TRRS, keebio-parts:TRRS-PJ-320A, symbol keebio:TRRS
- added U3: Pimoroni_trackpoint, Custom_footprints_Léon:Pimoroni_trackpoint, symbol Custom_symboles_Léon:Pimoroni_trackpoint
Connections:
- new net: D18.2 (A), MX18.2 (ROW)
- new net: D10.2 (A), MX10.2 (ROW)
- new net: D8.2 (A), MX8.2 (ROW)
- new net: D1.2 (A), MX1.2 (ROW)
- new net: D17.2 (A), MX17.2 (ROW)
- new net: D7.2 (A), MX7.2 (ROW)
- new net: RGB3.2 (DOUT), RGB4.4 (DIN)
- new net: RGB2.2 (DOUT), RGB3.4 (DIN)
- new net: D5.2 (A), MX5.2 (ROW)
- new net: D21.2 (A), MX21.2 (ROW)
- new net: D15.2 (A), MX15.2 (ROW)
- new net: D2.2 (A), MX2.2 (ROW)
- new net: D20.2 (A), MX20.2 (ROW), MX25.2 (ROW)
- new net: D12.2 (A), MX12.2 (ROW)
- new net: D14.2 (A), MX14.2 (ROW)
- new net: D16.2 (A), MX16.2 (ROW)
- new net: RGB1.2 (DOUT), RGB2.4 (DIN)
- new net: D3.2 (A), MX3.2 (ROW)
- new net: D13.2 (A), MX13.2 (ROW)
- new net: D22.2 (A), MX22.2 (ROW)
- new net: D9.2 (A), MX9.2 (ROW)
- new net: RGB5.2 (DOUT), RGB6.4 (DIN)
- new net: D23.2 (A), MX23.2 (ROW)
- new net: D19.2 (A), MX19.2 (ROW)
- new net: D6.2 (A), MX6.2 (ROW)
- new net: RGB4.2 (DOUT), RGB5.4 (DIN)
- new net: D4.2 (A), MX4.2 (ROW)
- new net: D11.2 (A), MX11.2 (ROW)
- new net COL0: MX1.1 (COL), MX2.1 (COL), MX3.1 (COL), MX4.1 (COL), U1.8 (5/C6)
- new net COL1: MX5.1 (COL), MX6.1 (COL), MX7.1 (COL), MX8.1 (COL), U1.18 (F6/A1)
- new net COL2: MX10.1 (COL), MX11.1 (COL), MX12.1 (COL), MX9.1 (COL), U1.17 (F7/A0)
- new net COL3: MX13.1 (COL), MX14.1 (COL), MX15.1 (COL), MX16.1 (COL), U1.16 (B1/15)
- new net COL4: MX17.1 (COL), MX18.1 (COL), MX19.1 (COL), MX20.1 (COL), MX25.1 (COL), U1.15 (B3/14)
- new net COL5: MX21.1 (COL), MX22.1 (COL), MX23.1 (COL), MX24.1 (COL), SW1.S2, U1.14 (B2/16)
- new net DATA: U1.1 (TX0/D3), U2.4 (RING2)
- new net ENC_A: SW1.A, U1.20 (F4/A3)
- new net ENC_B: SW1.B, U1.19 (F5/A2)
- new net ENC_S_A: D24.2 (A), MX24.2 (ROW), SW1.S1
- new net GND: RGB1.3 (VSS), RGB2.3 (VSS), RGB3.3 (VSS), RGB4.3 (VSS), RGB5.3 (VSS), RGB6.3 (VSS), SW1.C, U1.23 (GND), U1.3 (GND), U1.4 (GND), U2.1 (SLEEVE), U2.3 (RING1), U3.5 (GND)
- new net RGB: RGB1.4 (DIN), U1.2 (RX1/D2)
- new net ROW0_L: D1.1 (K), D13.1 (K), D17.1 (K), D21.1 (K), D5.1 (K), D9.1 (K), U1.7 (4/D4)
- new net ROW1_L: D10.1 (K), D14.1 (K), D18.1 (K), D2.1 (K), D22.1 (K), D6.1 (K), U1.13 (B6/10)
- new net ROW2_L: D11.1 (K), D15.1 (K), D19.1 (K), D23.1 (K), D3.1 (K), D7.1 (K), U1.10 (7/E6)
- new net ROW3_L: D12.1 (K), D16.1 (K), D20.1 (K), D24.1 (K), D4.1 (K), D8.1 (K), U1.11 (8/B4)
- new net SCL: U1.6 (3/D0/SCL), U3.3 (SCL)
- new net SDA: U1.5 (2/D1/SDA), U3.2 (SDA)
- new net VCC: RGB1.1 (VDD), RGB2.1 (VDD), RGB3.1 (VDD), RGB4.1 (VDD), RGB5.1 (VDD), RGB6.1 (VDD), U1.12 (9/B5), U1.21 (VCC), U2.2 (TIP), U3.1 (3-5V)
- no-connect marks 0 -> 1

Commit message: clean up
Parts:
- removed MX25: MX-NoLED, MX_Only:MXOnly-2U-ReversedStabilizers-NoLED, symbol MX_Alps_Hybrid:MX-NoLED
- added H1, H2, H3, H4, H5: MountingHole, MountingHole:MountingHole_2.1mm, symbol Mechanical:MountingHole
- added MX12.1, MX8.1: MX-NoLED, MX_Only:MXOnly-1U-NoLED, symbol MX_Alps_Hybrid:MX-NoLED
- added MX2.1: MX-NoLED, MX_Only:MXOnly-1.25U-NoLED, symbol MX_Alps_Hybrid:MX-NoLED
- added MX20.1: MX-NoLED, MX_Only:MXOnly-2U-ReversedStabilizers-NoLED, symbol MX_Alps_Hybrid:MX-NoLED
- U1: footprint kbd:ArduinoProMicro_centered -> Custom_footprints_Léon:ArduinoProMicro_centered
Connections:
- net COL0: now also MX2.1.1 (COL)
- net COL1: now also MX8.1.1 (COL)
- net COL2: now also MX12.1.1 (COL)
- net COL4: now also MX20.1.1 (COL)
- net at D8.2 (A), MX8.2 (ROW): now also MX8.1.2 (ROW)
- net at D2.2 (A), MX2.2 (ROW): now also MX2.1.2 (ROW)
- net at D20.2 (A), MX20.2 (ROW): now also MX20.1.2 (ROW)
- net at D12.2 (A), MX12.2 (ROW): now also MX12.1.2 (ROW)
Other:
- moved on the sheet: D1, D10, D11, D12, D13, D14, D15, D16, D17, D18, D19, D2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
