File: REV.1/chocobanan rev.1.kicad_pcb (KiCad board)
At the start: 2 copper layers, 158.9 x 100.2 mm, 92 parts, among them J1 USB_C_Receptacle_USB2.0, J2 Conn_01x05, J3 AudioJack4, SW1 SW_Push, SW2 SW_Push, U1 RP2040, U2 XC6206PxxxMR, U3 SRV05-4, U4 W25Q128JVS, Y1 Crystal_GND24

Commit message: safety commit
Parts:
- added LED10: WS2812B, Custom_footprints_Léon:XINGLIGHT_XL-1010RGBC-WS2812B, B.Cu at (132.9, 47.0)
- added LED11: WS2812B, Custom_footprints_Léon:XINGLIGHT_XL-1010RGBC-WS2812B, B.Cu at (129.9, 63.8)
- added LED12: WS2812B, Custom_footprints_Léon:XINGLIGHT_XL-1010RGBC-WS2812B, B.Cu at (127.0, 80.6)
- added LED13: WS2812B, Custom_footprints_Léon:XINGLIGHT_XL-1010RGBC-WS2812B, B.Cu at (110.2, 77.6)
- added LED14: WS2812B, Custom_footprints_Léon:XINGLIGHT_XL-1010RGBC-WS2812B, B.Cu at (89.1, 73.9)
- added LED15: WS2812B, Custom_footprints_Léon:XINGLIGHT_XL-1010RGBC-WS2812B, B.Cu at (56.2, 68.1)
- added LED16: WS2812B, Custom_footprints_Léon:XINGLIGHT_XL-1010RGBC-WS2812B, B.Cu at (36.2, 64.4)
- added LED17: WS2812B, Custom_footprints_Léon:XINGLIGHT_XL-1010RGBC-WS2812B, B.Cu at (136.0, 64.7)
- added LED18: WS2812B, Custom_footprints_Léon:XINGLIGHT_XL-1010RGBC-WS2812B, B.Cu at (136.0, 67.2)
- added LED7: WS2812B, Custom_footprints_Léon:XINGLIGHT_XL-1010RGBC-WS2812B, B.Cu at (109.4, 4.19)
- added LED8: WS2812B, Custom_footprints_Léon:XINGLIGHT_XL-1010RGBC-WS2812B, B.Cu at (109.4, 23.5)
- added LED9: WS2812B, Custom_footprints_Léon:XINGLIGHT_XL-1010RGBC-WS2812B, B.Cu at (106.1, 42.3)
- added U5: 74AHCT1G125, Package_TO_SOT_SMD:SOT-23-5, B.Cu at (-11.8, 0.00)
- J3: footprint keebio-parts:TRRS-PJ-320A -> Custom_footprints_Léon:CUI_SJ-43614-SMT
- LED1, LED2, LED3, LED4, LED5, LED6: footprint LED_SMD:LED_WS2812B_PLCC4_5.0x5.0mm_P3.2mm -> Custom_footprints_Léon:XINGLIGHT_XL-1010RGBC-WS2812B
- moved LED4 83.0 mm to (42.9, -7.53), turned to 175 degrees
- moved LED6 80.7 mm to (83.8, -0.31), turned to 170 degrees
- moved C1 74.9 mm to (0.00, 5.31), turned to 0 degrees
- moved U2 74.5 mm to (0.00, 7.47), turned to 180 degrees
- moved C2 74.2 mm to (0.00, 9.63), turned to 180 degrees
- moved LED3 72.1 mm to (22.2, -7.53), turned to 180 degrees
- moved C6 69.4 mm to (2.78, 7.47), turned to 90 degrees
- moved LED5 55.2 mm to (63.8, -3.84), turned to 170 degrees
- moved LED2 49.5 mm to (6.37, -7.53), turned to 180 degrees
- moved J2 42.2 mm to (23.8, 28.6), turned to 90 degrees
- moved SW2 40.7 mm to (89.6, 37.4), turned to 80 degrees
- moved LED1 31.6 mm to (-12.3, -7.53)
- moved J3 7.10 mm to (75.7, -12.8), turned to -100 degrees
- moved R7 3.45 mm to (83.3, 36.3), turned to 180 degrees
- moved R8 2.79 mm to (83.3, 35.1), turned to 0 degrees
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Connections:
- J2 pad 1: RESET -> GND
- J2 pad 2: SWD -> +3V3
- J2 pad 4: GND -> SWD
- J2 pad 5: +3V3 -> RESET
- J3 pad R1: GND -> +3V3
- J3 pad S: unconnected-(J3-PadS) -> GND
- J3 pad T: +3V3 -> GND
- LED1 pad 4: DATA -> RGB
- LED6 pad 2: unconnected-(LED6-DOUT-Pad2) -> Net-(LED6-DOUT)
- U1 pad 27: unconnected-(U1-GPIO16-Pad27) -> COL1
- U1 pad 28: unconnected-(U1-GPIO17-Pad28) -> ROW2
- U1 pad 29: unconnected-(U1-GPIO18-Pad29) -> RGBLED
- U1 pad 30: unconnected-(U1-GPIO19-Pad30) -> COL0
- U1 pad 31: unconnected-(U1-GPIO20-Pad31) -> ROW1
- U1 pad 32: unconnected-(U1-GPIO21-Pad32) -> ROW0
Routing:
- net +5V: track 150.7 -> 362.5 mm
- net RGBLED: track 0.00 -> 92.2 mm
- net COL0: track 58.9 -> 130.3 mm
- net ROW0: track 108.5 -> 179.7 mm, vias 2 -> 3
- net COL1: track 75.1 -> 146.0 mm
- net +3V3: track 54.8 -> 119.4 mm
- net ROW1: track 108.0 -> 171.9 mm
- net ROW2: track 110.1 -> 168.3 mm
- net GND: track 26.0 -> 58.8 mm, vias 14 -> 15
- net RESET: track 10.7 -> 41.4 mm
- net COL4: track 94.3 -> 65.8 mm
- net SWD: track 10.7 -> 38.7 mm
- net Net-(LED10-DIN): track 0.00 -> 26.7 mm
- net Net-(LED6-DOUT): track 0.00 -> 25.3 mm
- net SWC: track 10.7 -> 35.9 mm
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Other:
- outline, holes or cut-outs redrawn

Commit message: preparing for pc swap
Parts:
- removed the LED1 at (-12.3, -7.53)
- added LED19: WS2812B, Custom_footprints_Léon:XINGLIGHT_XL-1010RGBC-WS2812B, B.Cu at (-21.8, 45.6)
- added LED2: WS2812B, Custom_footprints_Léon:XINGLIGHT_XL-1010RGBC-WS2812B, B.Cu at (6.37, -7.53)
- added LED20: WS2812B, Custom_footprints_Léon:XINGLIGHT_XL-1010RGBC-WS2812B, B.Cu at (-21.8, 30.6)
- added LED21: WS2812B, Custom_footprints_Léon:XINGLIGHT_XL-1010RGBC-WS2812B, B.Cu at (-17.1, 11.5)
- MX20, MX21: footprint MX_Only:MXOnly-1.25U-NoLED -> MX_Only:MXOnly-1U-NoLED
- SW1, SW2: footprint Connector_PinHeader_2.54mm:PinHeader_1x02_P2.54mm_Vertical -> Button_Switch_SMD:SW_SPST_TL3342
- moved LED18 153.0 mm to (-17.1, 64.7)
- moved LED17 131.2 mm to (4.76, 64.7)
- moved SW1 103.6 mm to (19.1, 28.6)
- moved R5 66.3 mm to (13.1, -4.04), turned to -90 degrees
- moved R4 65.6 mm to (15.5, -4.04), turned to -90 degrees
- moved C4 65.3 mm to (15.0, 2.87), turned to 90 degrees
- moved C11 65.0 mm to (13.9, 2.87), turned to 90 degrees
- moved C3 62.4 mm to (12.3, 2.87), turned to 90 degrees
- moved C8 62.4 mm to (7.63, 6.92), turned to 180 degrees
- moved C7 62.3 mm to (10.9, 2.87), turned to 90 degrees
- moved C16 59.0 mm to (30.0, 6.92), turned to -90 degrees
- moved C9 54.5 mm to (7.63, 10.5), turned to 180 degrees
- moved U4 52.5 mm to (33.3, 9.52), turned to -90 degrees
- moved SW2 52.3 mm to (38.1, 28.6), turned to 0 degrees
- moved C13 51.3 mm to (20.9, 6.92), turned to 0 degrees
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- renumbered LED2 to LED1
Connections:
- J2 pad 1: GND -> SWC
- J2 pad 2: +3V3 -> SWD
- J2 pad 3: SWC -> RESET
- J2 pad 4: SWD -> GND
- J2 pad 5: RESET -> +3V3
- J3 pad R1: +3V3 -> GND
- J3 pad R2: serial -> GND
- J3 pad S: GND -> +3V3
- J3 pad T: GND -> serial
- LED1 pad 2: Net-(LED2-DOUT) -> Net-(LED1-DOUT)
- LED1 pad 4: Net-(LED1-DOUT) -> RGB
- LED18 pad 2: unconnected-(LED18-DOUT-Pad2) -> Net-(LED18-DOUT)
- MX19.1 pad A: unconnected-(MX19.1-PadA) -> ENC_A
- MX19.1 pad B: unconnected-(MX19.1-PadB) -> ENC_B
- MX19.1 pad C: unconnected-(MX19.1-PadC) -> GND
- U1 pad 11: unconnected-(U1-GPIO8-Pad11) -> COL3
- U1 pad 12: unconnected-(U1-GPIO9-Pad12) -> COL2
- U1 pad 13: unconnected-(U1-GPIO10-Pad13) -> COL1
- U1 pad 2: unconnected-(U1-GPIO0-Pad2) -> serial
- U1 pad 27: COL1 -> +3V3
- U1 pad 28: ROW2 -> COL0
- U1 pad 29: RGBLED -> ROW3
- U1 pad 3: unconnected-(U1-GPIO1-Pad3) -> ROW0
- U1 pad 30: COL0 -> RGBLED
- U1 pad 31: ROW1 -> unconnected-(U1-GPIO20-Pad31)
- U1 pad 32: ROW0 -> unconnected-(U1-GPIO21-Pad32)
- U1 pad 4: unconnected-(U1-GPIO2-Pad4) -> ENC_B
- U1 pad 5: unconnected-(U1-GPIO3-Pad5) -> ENC_A
- U1 pad 6: unconnected-(U1-GPIO4-Pad6) -> ROW2
- U1 pad 7: unconnected-(U1-GPIO5-Pad7) -> ROW1
- U1 pad 8: unconnected-(U1-GPIO6-Pad8) -> COL5
- U1 pad 9: unconnected-(U1-GPIO7-Pad9) -> COL4
Routing:
- net ENC_B: track 0.00 -> 153.1 mm
- net ENC_A: track 0.00 -> 147.8 mm
- net +5V: track 362.5 -> 508.0 mm, vias 4 -> 3
- net +3V3: track 119.4 -> 263.4 mm, vias 1 -> 4
- net COL4: track 65.8 -> 162.8 mm
- net COL5: track 66.1 -> 157.7 mm
- net ROW3: track 24.2 -> 109.9 mm
- net D+: track 93.3 -> 9.89 mm
- net D-: track 92.2 -> 9.89 mm
- net ROW2: track 168.3 -> 248.0 mm
- net serial: track 0.00 -> 75.8 mm, vias 0 -> 2
- net RGBLED: track 92.2 -> 23.9 mm
- net COL1: track 146.0 -> 87.7 mm
- net ROW1: track 171.9 -> 219.8 mm
- net COL3: track 82.8 -> 128.2 mm
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