File: REV.1/chocobanan rev.1.kicad_sch (KiCad schematic)
At the start: 92 parts, among them J1 USB_C_Receptacle_USB2.0, J2 Conn_01x05, J3 AudioJack4, SW1 SW_Push, SW2 SW_Push, U1 RP2040, U2 XC6206PxxxMR, U3 SRV05-4, U4 W25Q128JVS, Y1 Crystal_GND24

Commit message: safety commit
Parts:
- added LED10, LED11, LED12, LED13, LED14, LED15, LED16, LED17, LED18, LED7, LED8, LED9: WS2812B, Custom_footprints_Léon:XINGLIGHT_XL-1010RGBC-WS2812B, symbol LED:WS2812B
- added U5: 74AHCT1G125, Package_TO_SOT_SMD:SOT-23-5, symbol 74xGxx:74AHCT1G125
- C1: footprint keebio-parts:TRRS-PJ-320A-no-Fmask -> Capacitor_SMD:C_0402_1005Metric
- J3: footprint keebio-parts:TRRS-PJ-320A -> Custom_footprints_Léon:CUI_SJ-43614-SMT
- LED1, LED2, LED3, LED4, LED5, LED6: footprint LED_SMD:LED_WS2812B_PLCC4_5.0x5.0mm_P3.2mm -> Custom_footprints_Léon:XINGLIGHT_XL-1010RGBC-WS2812B
Connections:
- net +3V3: now also J2.2 (Pin_2), J3.R1; no longer J2.5 (Pin_5), J3.T
- net +5V: now also LED10.1 (VDD), LED11.1 (VDD), LED12.1 (VDD), LED13.1 (VDD), LED14.1 (VDD), LED15.1 (VDD), LED16.1 (VDD), LED17.1 (VDD), LED18.1 (VDD), LED7.1 (VDD), LED8.1 (VDD), LED9.1 (VDD), U5.5 (+5V)
- net COL0: now also U1.30 (GPIO19)
- net COL1: now also U1.27 (GPIO16)
- net GND: now also J2.1 (Pin_1), J3.S, J3.T, LED10.3 (VSS), LED11.3 (VSS), LED12.3 (VSS), LED13.3 (VSS), LED14.3 (VSS), LED15.3 (VSS), LED16.3 (VSS), LED17.3 (VSS), LED18.3 (VSS), LED7.3 (VSS), LED8.3 (VSS), LED9.3 (VSS), U5.1, U5.3 (GND); no longer J2.4 (Pin_4), J3.R1
- net RESET: now also J2.5 (Pin_5); no longer J2.1 (Pin_1)
- net ROW0: now also U1.32 (GPIO21)
- net ROW1: now also U1.31 (GPIO20)
- net ROW2: now also U1.28 (GPIO17)
- net SWD: now also J2.4 (Pin_4); no longer J2.2 (Pin_2)
- net RGBLED: now reaches U1.29 (GPIO18)
- net RGBLED: now also U5.2
- net at LED6.2 (DOUT): now also LED7.4 (DIN)
- net DATA renamed RGB
- net RGB: now also U5.4
- new net: LED10.4 (DIN), LED9.2 (DOUT)
- new net: LED8.2 (DOUT), LED9.4 (DIN)
- new net: LED11.2 (DOUT), LED12.4 (DIN)
- new net: LED10.2 (DOUT), LED11.4 (DIN)
- new net: LED14.2 (DOUT), LED15.4 (DIN)
- new net: LED13.2 (DOUT), LED14.4 (DIN)
- new net: LED12.2 (DOUT), LED13.4 (DIN)
- new net: LED7.2 (DOUT), LED8.4 (DIN)
- new net: LED17.2 (DOUT), LED18.4 (DIN)
- new net: LED16.2 (DOUT), LED17.4 (DIN)
- new net: LED15.2 (DOUT), LED16.4 (DIN)
- no-connect marks 6 -> 5
Other:
- moved on the sheet: LED1, LED2, LED3, LED4, LED5, LED6

Commit message: preparing for pc swap
Parts:
- removed LED1: WS2812B, Custom_footprints_Léon:XINGLIGHT_XL-1010RGBC-WS2812B, symbol LED:WS2812B
- added LED19, LED2, LED20, LED21: WS2812B, Custom_footprints_Léon:XINGLIGHT_XL-1010RGBC-WS2812B, symbol LED:WS2812B
- MX20, MX21: footprint MX_Only:MXOnly-1.25U-NoLED -> MX_Only:MXOnly-1U-NoLED
- SW1, SW2: footprint Connector_PinHeader_2.54mm:PinHeader_1x02_P2.54mm_Vertical -> Button_Switch_SMD:SW_SPST_TL3342
- renumbered LED2 to LED1
Connections:
- net +3V3: now also J2.5 (Pin_5), J3.S, U1.27 (GPIO16); no longer J2.2 (Pin_2), J3.R1
- net +5V: now also LED19.1 (VDD), LED2.1 (VDD), LED20.1 (VDD), LED21.1 (VDD)
- net COL0: now also U1.28 (GPIO17); no longer U1.30 (GPIO19)
- net COL1: now also U1.13 (GPIO10); no longer U1.27 (GPIO16)
- net COL2: now also U1.12 (GPIO9)
- net COL3: now also U1.11 (GPIO8)
- net COL4: now also U1.9 (GPIO7)
- net COL5: now also U1.8 (GPIO6)
- net GND: now also J2.4 (Pin_4), J3.R1, J3.R2, MX19.1.C, LED19.3 (VSS), LED2.3 (VSS), LED20.3 (VSS), LED21.3 (VSS); no longer J2.1 (Pin_1), J3.S, J3.T
- net RESET: now also J2.3 (Pin_3); no longer J2.5 (Pin_5)
- net RGB: now also LED1.4 (DIN)
- net RGBLED: now also U1.30 (GPIO19); no longer U1.29 (GPIO18)
- net ROW0: now also U1.3 (GPIO1); no longer U1.32 (GPIO21)
- net ROW1: now also U1.7 (GPIO5); no longer U1.31 (GPIO20)
- net ROW2: now also U1.6 (GPIO4); no longer U1.28 (GPIO17)
- net ROW3: now also U1.29 (GPIO18)
- net SWC: now also J2.1 (Pin_1); no longer J2.3 (Pin_3)
- net SWD: now also J2.2 (Pin_2); no longer J2.4 (Pin_4)
- net serial: now also J3.T, U1.2 (GPIO0); no longer J3.R2
- net at LED1.2 (DOUT): now also LED2.4 (DIN); no longer LED3.4 (DIN)
- net ENC_B: now reaches U1.4 (GPIO2)
- net ENC_B: now also MX19.1.B
- net ENC_A: now reaches U1.5 (GPIO3)
- net ENC_A: now also MX19.1.A
- net at LED18.2 (DOUT): now also LED19.4 (DIN)
- new net: LED20.2 (DOUT), LED21.4 (DIN)
- new net: LED19.2 (DOUT), LED20.4 (DIN)
- new net: LED2.2 (DOUT), LED3.4 (DIN)
Other:
- moved on the sheet: C14, C15, LED1, LED10, LED11, LED12, LED13, LED14, LED15, LED16, LED17, LED18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
